File: KiCad/main/main.kicad_pcb (KiCad board)
At the start: 2 copper layers, 88 x 90.3 mm, 37 parts, among them J1 Hexpansion-Connector, U1 TCA8418, U2 AP3032AKTR, U3 AT24CS02-MAHM

Commit message: fixed missing connections and changed eeprom
Parts:
- removed U3: AT24CS02-MAHM, Package_DFN_QFN:DFN-8-1EP_3x2mm_P0.5mm_EP1.3x1.5mm
- added R7: 3k3, Resistor_SMD:R_0603_1608Metric_Pad0.98x0.95mm_HandSolder, F.Cu at (-33.5, -36.8)
- added U4: AT24CS64-XHM, Package_SO:TSSOP-8_4.4x3mm_P0.65mm, F.Cu at (-15.4, -37.6)
Connections:
- J1 pad 19: !INT -> unconnected-(J1-HS_I-Pad19)
- J1 pad 2: unconnected-(J1-LS_A-Pad2) -> !INT
- J1 pad 3: unconnected-(J1-LS_B-Pad3) -> RST
- J1 pad 7: unconnected-(J1-LS_C-Pad7) -> LED_CTRL
- R5 pad 1: Net-(U2-CTRL) -> LED_CTRL
- U2 pad 4: Net-(U2-CTRL) -> LED_CTRL
Routing:
- net LED_CTRL: track 0.00 -> 71.4 mm, vias 0 -> 1
- net RST: track 11.8 -> 21.6 mm
- net VCC: track 119.7 -> 124.1 mm
- net Net-(U2-CTRL): track 3.38 -> 0.00 mm
- net !INT: track 26.6 -> 29.6 mm, vias 2 -> 1
- net GND: vias 12 -> 17

Commit message: Updated board designs to mirror hardware choices
Parts:
- U4: value AT24CS64-XHM -> ZD24C64A-XGMT

Commit message: _final_final_last_now_1
Parts:
- added J2: Conn_01x04_Socket, Connector_JST:JST_SH_SM04B-SRSS-TB_1x04-1MP_P1.00mm_Horizontal, F.Cu at (-40.4, -36.2)
- moved D1 6.95 mm to (-37.0, -43.5), turned to 90 degrees
- moved R1 6.84 mm to (-35.2, -43.5), turned to -90 degrees
Connections:
- J1 pad 12: unconnected-(J1-HS_F-Pad12) -> LED_CTRL
- J1 pad 18: unconnected-(J1-HS_H-Pad18) -> !INT
- J1 pad 2: !INT -> unconnected-(J1-LS_A-Pad2)
- J1 pad 7: LED_CTRL -> unconnected-(J1-LS_C-Pad7)
Routing:
- net SDA: track 25.6 -> 56.4 mm, vias 2 -> 4
- net SCL: track 26.1 -> 52.7 mm, vias 1 -> 3
- net !INT: track 29.6 -> 31.3 mm, vias 1 -> 2
- net VCC: track 124.1 -> 125.7 mm
- net /ROW6: track 122.9 -> 121.8 mm
- net LED_CTRL: track 71.4 -> 70.5 mm, vias 1 -> 2
- net GND: vias 17 -> 26
