File: KiCad/main/main.kicad_sch (KiCad schematic)
At the start: 37 parts, among them J1 Hexpansion-Connector, U1 TCA8418, U2 AP3032AKTR, U3 AT24CS02-MAHM

Commit message: fixed missing connections and changed eeprom
Parts:
- removed U3: AT24CS02-MAHM, Package_DFN_QFN:DFN-8-1EP_3x2mm_P0.5mm_EP1.3x1.5mm, symbol Memory_EEPROM:AT24CS02-MAHM
- added R7: 3k3, Resistor_SMD:R_0603_1608Metric_Pad0.98x0.95mm_HandSolder, symbol Device:R
- added U4: AT24CS64-XHM, Package_SO:TSSOP-8_4.4x3mm_P0.65mm, symbol Memory_EEPROM:AT24CS64-XHM
Connections:
- net !INT: now also J1.2 (LS_A), R7.1; no longer J1.19 (HS_I)
- net GND: now also U4.4 (GND)
- net RST: now also J1.3 (LS_B)
- net SCL: now also U4.6 (SCL)
- net SDA: now also U4.5 (SDA)
- net VCC: now also R7.2, U4.8 (VCC)
- net LED_CTRL: now reaches R5.1, U2.4 (CTRL)
- net LED_CTRL: now also J1.7 (LS_C)
- net at JP2.2 (B): now also U4.7 (WP)

Commit message: Updated board designs to mirror hardware choices
Parts:
- U4: value AT24CS64-XHM -> ZD24C64A-XGMT
Changed lines of the file:
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@@
 			)
 		)
-		(property "Value" "AT24CS64-XHM"
+		(property "Value" "ZD24C64A-XGMT"
 			(at 28.8133 172.72 0)
 			(effects
@@
 			)
 		)
-		(property "Datasheet" "http://ww1.microchip.com/downloads/en/DeviceDoc/Atmel-8870-SEEPROM-AT24CS64-Datasheet.pdf"
+		(property "Datasheet" ""
 			(at 26.67 180.34 0)
 			(effects
@@
 			)
 		)
-		(property "Description" "I2C Serial EEPROM, 64Kb (8192x8) with Unique Serial Number, TSSOP8"
+		(property "Description" ""
 			(at 26.67 180.34 0)
 			(effects

Commit message: _final_final_last_now_1
Parts:
- added J2: Conn_01x04_Socket, Connector_JST:JST_SH_SM04B-SRSS-TB_1x04-1MP_P1.00mm_Horizontal, symbol Connector:Conn_01x04_Socket
Connections:
- net !INT: now also J1.18 (HS_H); no longer J1.2 (LS_A)
- net GND: now also J2.1 (Pin_1)
- net LED_CTRL: now also J1.12 (HS_F); no longer J1.7 (LS_C)
- net SCL: now also J2.4 (Pin_4)
- net SDA: now also J2.3 (Pin_3)
- net VCC: now also J2.2 (Pin_2)
